File: board/sequencer_main.brd (EAGLE design)
At the start: 53.3 x 55.6 mm, 28 parts

Commit message: Added the proper board/schematic files for the circuit board. Inventor case files need to be rebuilt because inventor is stupid
Parts:
- moved C2 98.0 mm to (43.6, 24.5), turned to 180 degrees
- moved OSC_HEAD 86.3 mm to (43.7, 28.8)
- moved MUX_HEAD 74.2 mm to (23.6, 34.8), turned to 180 degrees
- moved CNTR_ARRAY 52.9 mm to (72.7, 42.2), flipped to the top, turned to 270 degrees
- moved R3 47.4 mm to (24.0, 43.1)
- moved C8 46.0 mm to (67.7, 29.5)
- moved R4 42.4 mm to (21.0, 43.3)
- moved R2 41.6 mm to (27.0, 42.9)
- moved EXT_OSC 40.5 mm to (72.8, 18.3), turned to 270 degrees
- moved C7 33.2 mm to (67.7, 24.5), turned to 0 degrees
- moved CNTR 32.9 mm to (64.3, 45.7), turned to 90 degrees
- moved C1 32.6 mm to (27.2, 26.5)
- moved POT_SW_ARRAY 31.9 mm to (32.7, 59.1)
- moved POT-MUX 28.9 mm to (34.6, 43.7)
- moved C6 25.9 mm to (33.0, 23.5), turned to 180 degrees
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Routing:
- net N$28: track 40.2 -> 4.15 mm
- net GND: track 115.1 -> 150.2 mm
- net N$52: track 8.68 -> 35.4 mm
- net N$50: track 16.6 -> 40.1 mm
- net VCC: track 106.9 -> 86.6 mm, vias 1 -> 0
- net N$9: track 17.4 -> 36.0 mm
- net N$38: track 44.4 -> 27.1 mm
- net N$12: track 9.31 -> 25.5 mm
- net N$11: track 22.6 -> 38.0 mm
- net N$10: track 20.5 -> 35.2 mm
- net N$43: track 14.0 -> 28.2 mm
- net N$40: track 0.00 -> 13.4 mm
- net N$47: track 39.4 -> 28.3 mm
- net N$48: track 15.4 -> 4.97 mm
- net N$51: track 36.9 -> 47.0 mm
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Other:
- board size 53.3 x 55.6 mm -> 55.8 x 51.5 mm
- board text added: "@lenord 2017"
- board text added: "ls-1"
- board text removed: "1"
- board text removed: "12"
- board text removed: "dtm 2017"
- board text removed: "ls-one sequencer"
